File: electronics/pcb/revB/design/VELOX_carrier_B.kicad_sch (KiCad schematic)
At the start: 45 parts, among them J1 Protected 1S cell, J2 RUN switch / OFF to charge, J3 USB-C charging only, J4 Solenoid, J5 RC522 keyed harness, J6 Buttons / LEDs / buzzer, Q1 AO3400A, Q2 AO3400A, U1 Arduino Nano ESP32, U2 4.2V charger / 100mA, U3 6V solenoid boost, U4 7.5V Nano boost, U5 USB overvoltage protector

Commit message: Complete Rev B routed PCB, native ERC/DRC checks and review package
Parts:
- added H1: M3 NPTH, VELOX:MountingHole_3.2mm_M3, symbol VELOX:Part_H1
- added H2: M3 NPTH, VELOX:MountingHole_3.2mm_M3, symbol VELOX:Part_H2
- added H3: M3 NPTH, VELOX:MountingHole_3.2mm_M3, symbol VELOX:Part_H3
- added H4: M3 NPTH, VELOX:MountingHole_3.2mm_M3, symbol VELOX:Part_H4
- C1: value 470u 10V -> 470u 10V / EEUFR1A471
- C10, C11: value 10u 25V -> 10u 25V X7R
- C8: value 100u 10V -> 100u 10V / EEUFR1A101
- C9: value 4.7u 50V -> 4.7u 50V X7R
- D3: value CHARGE LED -> CHARGE LED / red; footprint VELOX:LED_0805_2012Metric_Pad1.15x1.40mm_HandSolder -> VELOX:LED_0805_2012Metric
- F1: value 3A candidate fuse -> 3A / 0467003.NR candidate
- J1: value Protected 1S cell -> PROTECTED 1S BATTERY
- J2: value RUN switch / OFF to charge -> RUN SWITCH / OFF TO CHARGE
- J3: value USB-C charging only -> USB4125-GF-A / CHARGE ONLY; footprint Connector_USB:USB_C_Receptacle_GCT_USB4125-xx-x_6P_TopMnt_Horizontal -> VELOX:USB_C_Receptacle_GCT_USB4125-xx-x_6P_TopMnt_Horizontal
- J4: value Solenoid -> COIL / XH2 / 6V VERIFY
- J5: value RC522 keyed harness -> RC522 / XH8 HARNESS
- J6: value Buttons / LEDs / buzzer -> PANEL / PH8 HARNESS
- R11: value 10k 1% -> 10k 1% / 100mA
- R5, R6: value 220 -> 470
- TP1, TP2, TP3, TP4, TP5, TP6: now left out of the parts list
- U1: value Arduino Nano ESP32 -> Arduino Nano ESP32 ABX00083
- U2: value 4.2V charger / 100mA -> MCP73831-2ATI/OT; footprint VELOX:SOT-23-5 -> VELOX:SOT-23-5_HandSoldering
- U3: value 6V solenoid boost -> Pololu U3V40F6 / 6V; footprint VELOX:Pololu_4013_U3V40F6 -> VELOX:Pololu_U3V40F6_4013
- U4: value 7.5V Nano boost -> Pololu U3V16F7 / 7.5V; footprint VELOX:Pololu_4943_U3V16F7 -> VELOX:Pololu_U3V16F7_4943
- U5: value USB overvoltage protector -> NCP361SNT1G; footprint VELOX:SOT-23-5 -> VELOX:SOT-23-5_HandSoldering
Connections:
- net BAT_FUSED: now also C11.1, U2.3 (VBAT)
- net BAT_PROTECTED: no longer C11.1, U2.3 (VBAT)
- net CHARGE_LED_A renamed CHG_LED_A
- net CHARGE_PROG renamed CHG_PROG
- net CHARGE_STAT renamed CHG_STAT
- net USB_CC1 renamed CC1
- net USB_CC2 renamed CC2
Other:
- note added: "6 V COIL / SEPARATE FROM NANO VIN"
- note added: "90 x 55 mm / two layers. Not fabrication-released: battery, coil and enclosure must be qualified."
- note added: "BATTERY MONITOR"
- note added: "Battery must have independent protection. Flyback diode release delay and boost/battery pulse capability require real hardware tests."
- note added: "CONTROLLER / 3.3 V LOGIC"
- note added: "Charging: RUN switch open, Nano USB unplugged, verified cell temperature. No concurrent-use power path or cell-temperature cutoff."
- note added: "Matching labels connect. Nano ESP32 only; VBUS/B0/B1/D7 unused. Reader always powered: READER_POWER_GATED=0."
- note added: "PANEL / LEDS / BUZZER"
- note added: "Pololu modules use published top-view hole positions; no MT3608 or TP4056 clone interfaces."
- note added: "USB-C CHARGER / 100 mA / RUN OFF"
- note added: "VELOX CARRIER REV B | COMPACT ENGINEERING PROTOTYPE"
- note removed: "3.3V active buzzer / panel"
- note removed: "6V coil driver"
- note removed: "90 x 55 mm target. Copper routing and native ERC/DRC are unfinished. No manufacturing approval."
- note removed: "Battery monitor / calibrate ADC"
- note removed: "Nano ESP32 / 3.3V logic"
- note removed: "Power flags declare external supplies; they do not verify wiring. Polarity, coil load and enclosure fit require testing."
- note removed: "RC522: remote, always powered"
- note removed: "Same net labels connect. NC crosses are intentional. Charge with RUN OFF and Nano USB unplugged."
- note removed: "USB-C / OVP / 100mA charger"
- note removed: "Use a protected 1S cell. No onboard BMS, load sharing or temperature-qualified charging."
- note removed: "VELOX REV B | SCHEMATIC + PLACEMENT REVIEW | NOT FOR FABRICATION"
